File: Electronics/mainboard/mainboard.kicad_sch (KiCad schematic)
At the start: 18 parts, among them J1 CONN_P4_POWER_IN, J2 CONN_NIDEC_0, J3 CONN_NIDEC_1, J4 CONN_ESP32_L, J5 CONN_ESP32_R, J6 CONN_MPU6050, U3 LM7805_TO220

Commit message: assign footprints
Parts:
- removed J1: CONN_P4_POWER_IN, symbol Connector:Conn_01x02_Socket
- added C12: 100 nF, Capacitor_THT:C_Disc_D3.0mm_W2.0mm_P2.50mm, symbol Device:C
- added J7: Conn_Coaxial_Power, Connector_BarrelJack:BarrelJack_Horizontal, symbol Connector:Conn_Coaxial_Power
- C1: value C_Polarized -> 220 uF; footprint (none) -> Capacitor_THT:CP_Radial_D8.0mm_P3.50mm
- C10, C9: value C -> 47 nF; footprint (none) -> Capacitor_THT:C_Disc_D3.0mm_W2.0mm_P2.50mm
- C11, C7, C8: value C -> 100 nF; footprint (none) -> Capacitor_THT:C_Disc_D3.0mm_W2.0mm_P2.50mm
- C2, C3: value C_Polarized -> 470 uF; footprint (none) -> Capacitor_THT:CP_Radial_D10.0mm_P5.00mm
- C4: value C_Polarized -> 47 uF; footprint (none) -> Capacitor_THT:CP_Radial_D6.3mm_P2.50mm
- C5, C6: value C -> 330 nF; footprint (none) -> Capacitor_THT:C_Rect_L7.0mm_W2.5mm_P5.00mm
- J2, J3: footprint (none) -> Connector_JST:JST_EH_S8B-EH_1x08_P2.50mm_Horizontal
- J4, J5: footprint (none) -> Connector_PinHeader_2.54mm:PinHeader_1x08_P2.54mm_Vertical
- J6: footprint (none) -> Connector_PinHeader_2.54mm:PinHeader_1x06_P2.54mm_Vertical
Connections:
- net 3v3 is gone; now on net +3.3V: J4.1 (Pin_1)
- net 5v is gone; now on net +5V: J4.19 (Pin_19)
- net gnd is gone; now on net GND: J4.14 (Pin_14), J5.1 (Pin_1), J5.7 (Pin_7)
- net gpio16 is gone; now on net M0_ENC_A: J5.12 (Pin_12)
- net gpio17 is gone; now on net M0_ENC_V: J5.11 (Pin_11)
- net gpio18 is gone; now on net M0_PWM: J5.9 (Pin_9)
- net gpio19 is gone; now on net M0_BRK: J5.8 (Pin_8)
- net gpio21 is gone; now on net SDA_0: J5.6 (Pin_6)
- net gpio22 is gone; now on net SCL_0: J5.3 (Pin_3)
- net gpio25 is gone; now on net M0_DIR: J4.9 (Pin_9)
- net gpio26 is gone; now on net M0_PWM: J4.10 (Pin_10)
- net gpio27 is gone; now on net M0_BRK: J4.11 (Pin_11)
- net gpio32 is gone; now on net M0_ENC_A: J4.7 (Pin_7)
- net gpio33 is gone; now on net M0_ENC_V: J4.8 (Pin_8)
- net gpio35 is gone; now on net M0_ENC_B: J4.6 (Pin_6)
- net gpio4 is gone; now on net M0_ENC_B: J5.13 (Pin_13)
- net gpio5 is gone; now on net M0_DIR: J5.10 (Pin_10)
- net +5V: now reaches C9.1
- net +5V: now also C4.1, C7.1, U3.3 (VO), C12.1
- net GND: now reaches C9.2
- net GND: now also C1.2, C10.2, C11.2, C2.2, C3.2, C4.2, C5.2, C6.2, C7.2, C8.2, J2.2 (Pin_2), J3.2 (Pin_2), J6.2 (Pin_2), U3.2 (GND), C12.2, J7.2 (Ext)
- net +3.3V: now reaches C10.1
- net +3.3V: now also C11.1, C8.1, J6.1 (Pin_1)
- net +12V: now reaches C5.1
- net +12V: now also C1.1, C2.1, C3.1, C6.1, J2.1 (Pin_1), J3.1 (Pin_1), U3.1 (VI), J7.1 (In)
- net M0_BRK: now reaches J2.3 (Pin_3)
- net M0_BRK: now also J3.3 (Pin_3)
- net M0_PWM: now reaches J2.4 (Pin_4)
- net M0_PWM: now also J3.4 (Pin_4)
- net M0_DIR: now reaches J2.5 (Pin_5)
- net M0_DIR: now also J3.5 (Pin_5)
- net M0_ENC_V: now reaches J2.6 (Pin_6)
- net M0_ENC_V: now also J3.6 (Pin_6)
- net M0_ENC_A: now reaches J2.7 (Pin_7)
- net M0_ENC_A: now also J3.7 (Pin_7)
- net M0_ENC_B: now reaches J2.8 (Pin_8)
- net M0_ENC_B: now also J3.8 (Pin_8)
- net SCL_0: now reaches J6.3 (Pin_3)
- net SDA_0: now reaches J6.4 (Pin_4)
- net xda: now reaches J6.5 (Pin_5)
- net xcl: now reaches J6.6 (Pin_6)
- net ad0: now reaches J6.7 (Pin_7)
- net INT_0: now reaches J6.8 (Pin_8)
Other:
- moved on the sheet: C1, C10, C11, C2, C3, C4, C5, C6, C7, C8, C9, J2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

Commit message: export mainboard step
Parts:
- J4, J5: footprint Connector_PinHeader_2.54mm:PinHeader_1x08_P2.54mm_Vertical -> Connector_PinSocket_2.54mm:PinSocket_1x19_P2.54mm_Vertical
- J6: footprint Connector_PinHeader_2.54mm:PinHeader_1x06_P2.54mm_Vertical -> Connector_PinSocket_2.54mm:PinSocket_1x08_P2.54mm_Vertical
Connections:
- net M0_BRK: no longer J3.3 (Pin_3), J5.8 (Pin_8)
- net M0_DIR: no longer J3.5 (Pin_5), J5.10 (Pin_10)
- net M0_ENC_A: no longer J3.7 (Pin_7), J5.12 (Pin_12)
- net M0_ENC_B: no longer J3.8 (Pin_8), J5.13 (Pin_13)
- net M0_ENC_V: no longer J3.6 (Pin_6), J5.11 (Pin_11)
- net M0_PWM: no longer J3.4 (Pin_4), J5.9 (Pin_9)
- new net M1_BRK: J3.3 (Pin_3), J5.8 (Pin_8)
- new net M1_DIR: J3.5 (Pin_5), J5.10 (Pin_10)
- new net M1_ENC_A: J3.7 (Pin_7), J5.12 (Pin_12)
- new net M1_ENC_B: J3.8 (Pin_8), J5.13 (Pin_13)
- new net M1_ENC_V: J3.6 (Pin_6), J5.11 (Pin_11)
- new net M1_PWM: J3.4 (Pin_4), J5.9 (Pin_9)
Changed lines of the file:
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@@
 		)
 	)
-	(label "pwm"
+	(label "m0_pwm"
 		(at 59.69 92.71 180)
 		(effects
@@
 		)
 	)
-	(label "dir"
+	(label "m1_dir"
 		(at 59.69 129.54 180)
 		(effects
@@
 		)
 	)
-	(label "enc_vcc"
+	(label "e0_v+"
 		(at 59.69 97.79 180)
 		(effects
@@
 		)
 	)
-	(label "enc_vcc"
+	(label "e1_v+"
 		(at 59.69 132.08 180)
 		(effects
@@
 		)
 	)
-	(label "enc_b"
+	(label "e1_b"
 		(at 59.69 137.16 180)
 		(effects
@@
 		)
 	)
-	(label "brake"
+	(label "m0_brk"
 		(at 59.69 90.17 180)
 		(effects
@@
 		)
 	)
-	(label "enc_a"
+	(label "e0_a"
 		(at 59.69 100.33 180)
 		(effects
@@
 		)
 	)
-	(label "enc_a"
+	(label "e1_a"
 		(at 59.69 134.62 180)
 		(effects
@@
 		)
 	)
-	(label "pwm"
+	(label "m1_pwm"
 		(at 59.69 127 180)
 		(effects
@@
 		)
 	)
-	(label "brake"
+	(label "m1_brk"
 		(at 59.69 124.46 180)
 		(effects
@@
 		)
 	)
-	(label "enc_b"
+	(label "e0_b"
 		(at 59.69 102.87 180)
 		(effects
@@
 		)
 	)
-	(label "dir"
+	(label "m0_dir"
 		(at 59.69 95.25 180)
 		(effects
@@
 			)
 		)
-		(property "Footprint" "Connector_PinHeader_2.54mm:PinHeader_1x08_P2.54mm_Vertical"
+		(property "Footprint" "Connector_PinSocket_2.54mm:PinSocket_1x19_P2.54mm_Vertical"
 			(at 142.24 105.41 0)
 			(effects
@@
 			)
 		)
-		(property "Footprint" "Connector_PinHeader_2.54mm:PinHeader_1x08_P2.54mm_Vertical"
+		(property "Footprint" "Connector_PinSocket_2.54mm:PinSocket_1x19_P2.54mm_Vertical"
 			(at 163.83 105.41 0)
 			(effects
@@
 			)
 		)
-		(property "Footprint" "Connector_PinHeader_2.54mm:PinHeader_1x06_P2.54mm_Vertical"
+		(property "Footprint" "Connector_PinSocket_2.54mm:PinSocket_1x08_P2.54mm_Vertical"
 			(at 251.46 140.97 0)
 			(effects
